File: Boards-2024/2024.0/GHOUL-2024-0/GHOUL-2024-0.kicad_sch (KiCad schematic)
At the start: 76 parts, among them J1 USB_C_Receptacle_USB2.0, J2 U.FL, J3 SOICbite, J4 Conn_01x03_Pin, Q1 Q_NMOS_GSD, SW2 SLIDE, U1 MCU_RaspberryPi_RP2040_RP2040, U11 MAX-M10S, U2 TVS1800DRVR, U3 USBLC6-2SC6, U4 TPS2121RUXR, U5 W25Q128JVS, U6 LT6703CDC-3, U7 DRF1262TL, U8 MB85RS1MT, U9 MS5607-02BA, Y1 12MHz

Commit message: added notes to GHOUL 2024.0
Parts:
- added C24, C27: 15uF, Capacitor_SMD:C_1206_3216Metric, symbol Device:C_Small
- added L1, L2: 3.3uH, Inductor_SMD:L_1210_3225Metric, symbol Device:L_Small
- added R20, R21: 100m, Resistor_SMD:R_0603_1608Metric, symbol Device:R_Small
- R10, R8: value 5K -> ??
- R7, R9: value 23.7K -> ??
Connections:
- net +3V3: now also C27.1, L2.1, R21.1
- net +5V: now also C24.1, L1.1, R20.1
- net GND: now also C24.2, C27.2
- new net: L2.2, R21.2
- new net: L1.2, R20.2
- new net: U11.10 (GND), U11.12 (GND)
- no-connect marks 22 -> 28
Other:
- note added: "OV resistor values need checking"
- note added: "Power Filters to use"
- note added: "TODO: - Logic Power (3.3v and 5v) - Cutdown Power"
- note added: "U.FL for now but we probably have space for SMA"
