File: Boards-2024/2024.0/GHOUL-2024-0/GHOUL-2024-0.kicad_pcb (KiCad board)
At the start: 4 copper layers, 47 x 71 mm, 115 parts, among them J1 USB_C_Receptacle_USB2.0, J10 Conn_01x04, J2 U.FL, J3 SOICbite, J4 Conn_01x03_Pin, J5 Conn_01x04, J6 Conn_01x03, J7 Conn_01x02, J8 Conn_01x02, J9 Conn_01x04, Q1 Q_NMOS_GSD, Q2 Q_NMOS_GSD, Q3 Q_NMOS_GSD, Q4 Q_NMOS_GSD, Q5 Q_NMOS_GSD, Q6 Q_NMOS_GSD, Q7 Q_NMOS_GSD, SW2 SLIDE, U1 MCU_RaspberryPi_RP2040_RP2040, U10 LTM4622AEV-PBF, U11 MAX-M10S, U2 TVS1800DRVR, U3 USBLC6-2SC6, U4 TPS2121RUXR, U5 W25Q128JVS, U6 LT6703CDC-3, U7 DRF1262TL, U8 MB85RS1MT, U9 MS5607-02BA, Y1 12MHz

Commit message: your mom
Routing:
- net +5V: track 82.6 -> 90.4 mm, vias 5 -> 6
Changed lines of the file:
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@@
         (effects (font (size 1 1) (thickness 0.15)))
     )
-    (fp_text user "A" (at -3.75 -2.96 90 unlocked) (layer "F.SilkS")
+    (fp_text user "A" (at -4.27 -3.6 90 unlocked) (layer "F.SilkS")
         (effects (font (size 0.5 0.5) (thickness 0.125)))
     )
@@
         (effects (font (size 0.5 0.5) (thickness 0.125)))
     )
-    (fp_text user "E" (at -3.75 3.14 90 unlocked) (layer "F.SilkS")
+    (fp_text user "E" (at -3.62 3.83 90 unlocked) (layer "F.SilkS")
         (effects (font (size 0.5 0.5) (thickness 0.125)))
     )
-    (fp_text user "1" (at -2.8 -3.76 180 unlocked) (layer "F.SilkS")
+    (fp_text user "1" (at -2.68 -4.21 180 unlocked) (layer "F.SilkS")
         (effects (font (size 0.5 0.5) (thickness 0.125)))
     )
@@
   (segment (start 152.595 107.39) (end 151.205 108.78) (width 0.6) (layer "F.Cu") (net 13))
   (segment (start 149.81 106.1) (end 148.9 105.19) (width 0.2) (layer "F.Cu") (net 13))
-  (via (at 142.83 99.33) (size 0.75) (drill 0.6) (layers "F.Cu" "B.Cu") (net 13))
+  (via (at 142.27 98.95) (size 1) (drill 0.85) (layers "F.Cu" "B.Cu") (net 13))
   (via (at 148.9 105.19) (size 0.75) (drill 0.6) (layers "F.Cu" "B.Cu") (net 13))
   (via (at 151.59 106.68) (size 0.75) (drill 0.6) (layers "F.Cu" "B.Cu") (net 13))
   (via (at 146.81 102.79) (size 1) (drill 0.85) (layers "F.Cu" "B.Cu") (net 13))
   (via (at 150.68 105.21) (size 0.75) (drill 0.6) (layers "F.Cu" "B.Cu") (net 13))
-  (segment (start 142.59 99.57) (end 142.59 102.05) (width 0.75) (layer "In2.Cu") (net 13))
-  (segment (start 143.03 115.238629) (end 143.03 115.120972) (width 0.75) (layer "In2.Cu") (net 13))
-  (segment (start 147.93 110.220972) (end 147.93 105.47) (width 0.75) (layer "In2.Cu") (net 13))
-  (segment (start 136.685 139.685) (end 138.13 141.13) (width 0.75) (layer "In2.Cu") (net 13))
-  (segment (start 142.59 102.05) (end 144.26 103.72) (width 0.75) (layer "In2.Cu") (net 13))
-  (segment (start 143.08 115.951371) (end 143.08 115.288629) (width 0.75) (layer "In2.Cu") (net 13))
-  (segment (start 143.03 115.120972) (end 147.93 110.220972) (width 0.75) (layer "In2.Cu") (net 13))
-  (segment (start 138.13 132.23) (end 136.685 133.675) (width 0.75) (layer "In2.Cu") (net 13))
-  (segment (start 138.08 93.85) (end 140.96 93.85) (width 0.75) (layer "In2.Cu") (net 13))
-  (segment (start 143.08 115.288629) (end 143.03 115.238629) (width 0.75) (layer "In2.Cu") (net 13))
-  (segment (start 141.8 128.56) (end 141.8 122.62) (width 0.75) (layer "In2.Cu") (net 13))
-  (segment (start 142.83 99.33) (end 142.59 99.57) (width 0.75) (layer "In2.Cu") (net 13))
-  (segment (start 136.685 133.675) (end 136.685 139.685) (width 0.75) (layer "In2.Cu") (net 13))
-  (segment (start 142.83 95.72) (end 142.83 99.33) (width 0.75) (layer "In2.Cu") (net 13))
-  (segment (start 141.8 122.62) (end 143.03 121.39) (width 0.75) (layer "In2.Cu") (net 13))
-  (segment (start 143.03 121.39) (end 143.03 116.001371) (width 0.75) (layer "In2.Cu") (net 13))
-  (segment (start 140.96 93.85) (end 142.83 95.72) (width 0.75) (layer "In2.Cu") (net 13))
-  (segment (start 144.26 103.72) (end 144.83 103.72) (width 0.75) (layer "In2.Cu") (net 13))
-  (segment (start 138.13 132.23) (end 141.8 128.56) (width 0.75) (layer "In2.Cu") (net 13))
-  (segment (start 143.03 116.001371) (end 143.08 115.951371) (width 0.75) (layer "In2.Cu") (net 13))
+  (via (at 147.65 104.11) (size 0.8) (drill 0.4) (layers "F.Cu" "B.Cu") (free) (net 13))
+  (segment (start 136.23 134.13) (end 136.23 139.23) (width 1) (layer "In2.Cu") (net 13))
+  (segment (start 147.93 105.47) (end 148.62 105.47) (width 1) (layer "In2.Cu") (net 13))
+  (segment (start 143.31 121.11) (end 143.31 117.280491) (width 1) (layer "In2.Cu") (net 13))
+  (segment (start 147.65 104.11) (end 147.65 105.19) (width 0.6) (layer "In2.Cu") (net 13))
+  (segment (start 138.13 132.23) (end 136.23 134.13) (width 1) (layer "In2.Cu") (net 13))
+  (segment (start 138.13 132.23) (end 141.8 128.56) (width 1) (layer "In2.Cu") (net 13))
+  (segment (start 136.23 139.23) (end 138.13 141.13) (width 1) (layer "In2.Cu") (net 13))
+  (segment (start 141.8 128.56) (end 141.8 122.62) (width 1) (layer "In2.Cu") (net 13))
+  (segment (start 142.27 95.16) (end 140.96 93.85) (width 1) (layer "In2.Cu") (net 13))
+  (segment (start 142.27 101.37) (end 143.69 102.79) (width 1) (layer "In2.Cu") (net 13))
+  (segment (start 140.96 93.85) (end 138.08 93.85) (width 1) (layer "In2.Cu") (net 13))
+  (segment (start 147.65 105.19) (end 147.93 105.47) (width 0.6) (layer "In2.Cu") (net 13))
+  (segment (start 142.27 98.95) (end 142.27 95.16) (width 1) (layer "In2.Cu") (net 13))
+  (segment (start 142.27 98.95) (end 142.27 101.37) (width 1) (layer "In2.Cu") (net 13))
+  (segment (start 147.93 112.660491) (end 147.93 105.47) (width 1) (layer "In2.Cu") (net 13))
+  (segment (start 143.69 102.79) (end 146.81 102.79) (width 1) (layer "In2.Cu") (net 13))
+  (segment (start 150.66 105.19) (end 150.68 105.21) (width 0.2) (layer "In2.Cu") (net 13))
+  (segment (start 148.62 105.47) (end 148.9 105.19) (width 1) (layer "In2.Cu") (net 13))
+  (segment (start 148.9 105.19) (end 150.66 105.19) (width 1) (layer "In2.Cu") (net 13))
+  (segment (start 141.8 122.62) (end 143.31 121.11) (width 1) (layer "In2.Cu") (net 13))
+  (segment (start 143.31 117.280491) (end 147.93 112.660491) (width 1) (layer "In2.Cu") (net 13))
+  (segment (start 141.34 104.255) (end 141.47 104.385) (width 0.6) (layer "B.Cu") (net 13))
   (segment (start 141.515 104.34) (end 141.515 104.39) (width 1) (layer "B.Cu") (net 13))
   (segment (start 144.77 102.79) (end 143.065 102.79) (width 1) (layer "B.Cu") (net 13))
   (segment (start 141.465 104.39) (end 141.47 104.385) (width 0.45) (layer "B.Cu") (net 13))
   (segment (start 144.77 102.79) (end 146.81 102.79) (width 1) (layer "B.Cu") (net 13))
-  (segment (start 141.47 100.69) (end 142.83 99.33) (width 0.6) (layer "B.Cu") (net 13))
+  (segment (start 147.65 104.11) (end 147.65 103.63) (width 0.6) (layer "B.Cu") (net 13))
   (segment (start 141.905 106.44) (end 143.66 106.44) (width 0.6) (layer "B.Cu") (net 13))
   (segment (start 141.465 106) (end 141.905 106.44) (width 0.6) (layer "B.Cu") (net 13))
+  (segment (start 141.34 99.88) (end 141.34 104.255) (width 0.6) (layer "B.Cu") (net 13))
   (segment (start 143.66 106.44) (end 144.77 105.33) (width 0.6) (layer "B.Cu") (net 13))
+  (segment (start 141.47 99.75) (end 141.34 99.88) (width 0.6) (layer "B.Cu") (net 13))
   (segment (start 144.77 105.33) (end 144.77 102.79) (width 1.5) (layer "B.Cu") (net 13))
-  (segment (start 141.47 104.385) (end 141.47 100.69) (width 0.6) (layer "B.Cu") (net 13))
+  (segment (start 147.65 103.63) (end 146.81 102.79) (width 0.6) (layer "B.Cu") (net 13))
+  (segment (start 142.27 98.95) (end 141.47 99.75) (width 0.75) (layer "B.Cu") (net 13))
   (segment (start 143.065 102.79) (end 141.515 104.34) (width 1) (layer "B.Cu") (net 13))
   (segment (start 149.12 130.78) (end 149.59 131.25) (width 0.2) (layer "F.Cu") (net 14))
@@
   )
   (zone (net 2) (net_name "GND") (layers "F.Cu" "In1.Cu" "In2.Cu" "B.Cu") (hatch edge 0.5)
+    (priority 1)
     (connect_pads yes (clearance 0.127))
     (min_thickness 0.25) (filled_areas_thickness no)
@@
         (xy 156.59 126.67)
         (xy 164.080964 126.67)
-        (xy 164.080964 126.67)
         (xy 164.052159 136.23)

Commit message: did your mom
Routing:
- added copper zone on F.Cu, net Net-(C26-Pad1)
Changed lines of the file:
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@@
   (segment (start 146.205348 117.09) (end 143.334652 117.09) (width 0.2) (layer "B.Cu") (net 109))
   (segment (start 143.334652 117.09) (end 142.28 118.144652) (width 0.2) (layer "B.Cu") (net 109))
+  (zone (net 92) (net_name "Net-(C26-Pad1)") (layer "F.Cu") (hatch edge 0.5)
+    (priority 14)
+    (connect_pads yes (clearance 0.127))
+    (min_thickness 0.25) (filled_areas_thickness no)
+    (fill yes (thermal_gap 0.5) (thermal_bridge_width 0.5))
+    (polygon
+      (pts
+        (xy 152.06 102.11)
+        (xy 154.32 102.11)
+        (xy 154.42 102.21)
+        (xy 154.42 103.1)
+        (xy 154.06 103.46)
+        (xy 153.35 103.46)
+        (xy 153.35 104.82)
+        (xy 154.39 105.86)
+        (xy 154.39 108.78)
+        (xy 153.62 109.55)
+        (xy 152.33 109.55)
+        (xy 152.03 109.25)
+        (xy 152.03 108.26)
+        (xy 153.15 107.14)
+        (xy 153.15 105.92)
+        (xy 152.69 105.46)
+        (xy 151.82 105.46)
+        (xy 151.8 105.48)
+        (xy 151.38 105.06)
+        (xy 151.38 104.38)
+        (xy 148.43 104.38)
+        (xy 148.35 104.46)
+        (xy 148.27 104.38)
+        (xy 148.27 103.1)
+        (xy 148.51 102.86)
+        (xy 151.31 102.86)
+      )
+    )
+  )
   (zone (net 10) (net_name "VBUS") (layer "F.Cu") (hatch edge 0.5)
     (priority 8)
