File: Boards-2024/2024.0/GHOUL-2024-0/GHOUL-2024-0.kicad_pcb (KiCad board)
At the start: 4 copper layers, 47 x 71 mm, 115 parts, among them J1 USB_C_Receptacle_USB2.0, J10 Conn_01x04, J2 U.FL, J3 SOICbite, J4 Conn_01x03_Pin, J5 Conn_01x04, J6 Conn_01x03, J7 Conn_01x02, J8 Conn_01x02, J9 Conn_01x04, Q1 Q_NMOS_GSD, Q2 Q_NMOS_GSD, Q3 Q_NMOS_GSD, Q4 Q_NMOS_GSD, Q5 Q_NMOS_GSD, Q6 Q_NMOS_GSD, Q7 Q_NMOS_GSD, SW2 SLIDE, U1 MCU_RaspberryPi_RP2040_RP2040, U10 LTM4622AEV-PBF, U11 MAX-M10S, U2 TVS1800DRVR, U3 USBLC6-2SC6, U4 TPS2121RUXR, U5 W25Q128JVS, U6 LT6703CDC-3, U7 DRF1262TL, U8 MB85RS1MT, U9 MS5607-02BA, Y1 12MHz

Commit message: ordered GHOUL 2024.0
Parts:
- moved C32 0.09 mm to (149.5, 100.4)
Routing:
- net Net-(U10-FB2): track 3.41 -> 4.87 mm, vias 0 -> 2
- net Net-(U10-PG00D2): track 7.61 -> 6.20 mm, vias 0 -> 1
- net Net-(U10-TRACK/SS2): track 2.36 -> 3.55 mm, vias 0 -> 2
- net +3V3: track 105.5 -> 106.5 mm
- net Net-(U10-FREQ): track 5.09 -> 5.27 mm, vias 0 -> 2
Other:
- board text added: "Akemi & Shipman"
- board text added: "Akemi did this"
- board text added: "GHOUL 02/2024"
- board text added: "JLCJLCJLC"
- board text added: "flowbusters"
- board text added: "venting makes me feel good"
