File: Test-Cutdown-Board/Cutdown_Test/Cutdown_Test.kicad_pcb (KiCad board)
At the start: 4 copper layers, 27.5 x 34.1 mm, 32 parts, among them J1 Nichrome, J2 Conn_01x02_Socket, SW1 SW_SPDT, U1 LT3120JV-PBF

Commit message: minor cutdown circuit tuning
Routing:
- net GND: track 24.1 -> 25.6 mm, vias 6 -> 7
Changed lines of the file:
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@@
     (property "ki_keywords" "capacitor cap")
     (attr smd)
-    (fp_text reference "C2" (at 0 -1.1) (layer "F.SilkS")
+    (fp_text reference "C2" (at -0.4375 -1.1) (layer "F.SilkS")
         (effects (font (size 0.5 0.5) (thickness 0.125)))
     )
@@
   (segment (start 137.5 112.7375) (end 137.2375 112.7375) (width 0.25) (layer "F.Cu") (net 2))
   (segment (start 148.698101 102.44) (end 148.698101 101.098101) (width 1) (layer "F.Cu") (net 2))
+  (segment (start 142 103.9) (end 142 102.7) (width 0.5) (layer "F.Cu") (net 2))
   (segment (start 135.5 109.5) (end 135.05 109.05) (width 0.25) (layer "F.Cu") (net 2))
   (segment (start 135.5 110.4) (end 135.5 111) (width 0.25) (layer "F.Cu") (net 2))
@@
   (segment (start 133.6 114.9) (end 131.4875 114.9) (width 0.5) (layer "F.Cu") (net 2))
   (segment (start 134.3 114.5125) (end 133.9875 114.5125) (width 0.5) (layer "F.Cu") (net 2))
+  (segment (start 142 102.7) (end 141.8 102.5) (width 0.5) (layer "F.Cu") (net 2))
   (segment (start 148.698101 101.098101) (end 148.6 101) (width 1) (layer "F.Cu") (net 2))
   (segment (start 133.9875 114.5125) (end 133.6 114.9) (width 0.5) (layer "F.Cu") (net 2))
@@
   (via (at 140.4 114.5) (size 0.8) (drill 0.4) (layers "F.Cu" "B.Cu") (net 2))
   (via (at 132.7 114.9) (size 0.8) (drill 0.4) (layers "F.Cu" "B.Cu") (net 2))
+  (via (at 141.8 102.5) (size 0.8) (drill 0.4) (layers "F.Cu" "B.Cu") (net 2))
   (via (at 148.6 101) (size 0.8) (drill 0.4) (layers "F.Cu" "B.Cu") (net 2))
   (via (at 136 111.5) (size 0.8) (drill 0.4) (layers "F.Cu" "B.Cu") (net 2))
