File: Babel_Fish/Babel_Fish/Babel_Fish.kicad_sch (KiCad schematic)
At the start: 97 parts, among them J1 USB_C_Receptacle_USB2.0, J2 U.FL, J3 Conn_01x08, Q1 Q_NMOS_GSD, SW2 SLIDE, U1 MCU_RaspberryPi_RP2040_RP2040, U10 LT8653SIV-PBF, U2 TVS1800DRVR, U3 USBLC6-2SC6, U4 TPS2121RUXR, U5 W25Q128JVS, U6 LT6703CDC-3, U7 DRF1262TL, U8 MB85RS1MT, U9 WE 171010550, Y1 12MHz

Commit message: Babel Fish ready for layout
Parts:
- removed C27, C36: 470pF, Capacitor_SMD:C_0603_1608Metric, symbol Device:C_Small
- removed C28: 100nF, Capacitor_SMD:C_0603_1608Metric, symbol Device:C_Small
- removed C30, C34: 4.7pF, Capacitor_SMD:C_0603_1608Metric, symbol Device:C_Small
- removed C31, C33: 10nF, Capacitor_SMD:C_0603_1608Metric, symbol Device:C_Small
- removed C32: 1uF, Capacitor_SMD:C_0603_1608Metric, symbol Device:C_Small
- removed C38: 47uF, Capacitor_SMD:C_1206_3216Metric, symbol Device:C_Small
- removed L2, L3: 2.2uH, Inductor_SMD:L_1210_3225Metric, symbol Device:L_Small
- removed R23: 15K, Resistor_SMD:R_0603_1608Metric, symbol Device:R_Small
- removed R26: 100K, Resistor_SMD:R_0603_1608Metric, symbol Device:R_Small
- removed R27: 34.8K, Resistor_SMD:R_0603_1608Metric, symbol Device:R_Small
- removed U10: LT8653SIV-PBF, BITSv5:LT8653SIV-PBF, symbol BITSv5:LT8653SIV-PBF
- added H4: M2, MountingHole:MountingHole_2.2mm_M2_Pad, symbol Mechanical:MountingHole
- added J4: Conn_01x02, Connector_PinHeader_2.54mm:PinHeader_1x02_P2.54mm_Vertical, symbol Connector_Generic:Conn_01x02
- added U10: WE_171021801, BPP_Lib:WE_171021801, symbol BPP_Lib:WE_171021801
- C25: value 47uF -> DNF; footprint Capacitor_SMD:C_1206_3216Metric -> Capacitor_SMD:C_0805_2012Metric
- C26: value 4.7uF -> DNF; footprint Capacitor_SMD:C_0603_1608Metric -> Capacitor_SMD:C_0805_2012Metric
- C29: value ??uF -> 22pF; footprint (none) -> Capacitor_SMD:C_0603_1608Metric
- C35: value ??uF -> 10uF; footprint (none) -> Capacitor_SMD:C_0805_2012Metric
- C37: value ??uF -> 4.7uF; footprint (none) -> Capacitor_SMD:C_0805_2012Metric
- J3: footprint (none) -> Connector_PinHeader_2.54mm:PinHeader_1x08_P2.54mm_Vertical
- JP1, JP2: footprint (none) -> Jumper:SolderJumper-2_P1.3mm_Open_TrianglePad1.0x1.5mm
- R18: value ??k -> 100k; footprint (none) -> Resistor_SMD:R_0603_1608Metric
- R19: value ??k -> 32.4k; footprint (none) -> Resistor_SMD:R_0603_1608Metric
- R21: value 22.1K -> 10k
- R22: value 100K -> 1.87k
- SW1: footprint BITSv5:CAS-120TB_NDC-M -> BPP_Lib:CAS-120TB_NDC-M
- SW2: footprint BITSv5:CL-SB-12B-01_NDC -> BPP_Lib:CL-SB-12B-01_NDC
- U1: footprint BITSv5:RP2040-QFN-56 -> BPP_Lib:RP2040-QFN-56
- U2: footprint BITSv5:TVS1800 -> BPP_Lib:TVS1800
- U3: footprint BITSv5:SOT23-6L_STM -> Package_TO_SOT_SMD:SOT-23-6
- U4: footprint BITSv5:TPS2121 -> BPP_Lib:TPS2121
- U5: footprint BITSv5:WSON_128JVPIQ_WIN -> BPP_Lib:W25Q64JVZP
- U6: footprint BITSv5:DFN-3_DC_LIT -> BPP_Lib:DFN-3_DC_LIT
- U7: footprint BITSv5:DRF1262TL -> BPP_Lib:DRF1262TL
- U9: footprint (none) -> BPP_Lib:WE_171010550
Connections:
- net VCC is gone; now on net +BATT: C19.1, R15.1, R17.1, U6.2 (V+)
- net +3V3: no longer C29.1, C35.1, R18.1, U9.6 (VOUT)
- net +5V: now also J4.1 (Pin_1)
- net +BATT: now also C26.1, U10.1 (VIN), U10.2 (VIN), U10.3 (VIN), U10.4 (VIN)
- net GND: now also R22.2, U5.9 (GND), U9.EP (PGND), J4.2 (Pin_2), U10.EP (PGND)
- net VBUS: now also J1.A4 (VBUS), J1.A9 (VBUS), J1.B4 (VBUS), J1.B9 (VBUS), U3.5
- net at R21.1: now also C10.1, C25.1, R9.1, U4.2 (IN2), U10.10 (VOUT), U10.11 (VOUT), U10.12 (VOUT), U10.9 (VOUT)
- net at L4.2, R29.2: now also C29.1, C35.1, R18.1, U9.6 (VOUT)
- net at C17.1, U4.1 (OUT), U4.8 (OUT): now also L1.2, R20.2
- net at R21.2: now also R22.1, U10.13 (FB)
- net LVC_CUTOFF renamed CUTOFF
- net CUTOFF: now also U10.16 (EN)
- new net: U10.14 (NC), U10.15 (NC), U10.5 (NC), U10.6 (NC), U10.7 (NC), U10.8 (NC)
- no-connect marks 15 -> 12
Other:
- note added: "3.3v Regulator"
- note added: "5v Regulator"
- note removed: "5V / 3.3V Buck Regulator"
- moved on the sheet: C10, C16, C17, C19, C24, C29, C35, C37, C39, C9, H1, H2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

Commit message: started routing Babel Fish
Parts:
- added J5: Conn_01x04, Connector_PinHeader_2.54mm:PinHeader_1x04_P2.54mm_Vertical, symbol Connector_Generic:Conn_01x04
Connections:
- net +3V3: now also J5.1 (Pin_1)
- net GND: now also J5.4 (Pin_4)
- net SCL: now also J5.3 (Pin_3)
- net SDA: now also J5.2 (Pin_2)
- net EXTINT: no longer names the net of U1.28 (GPIO17)
- net TIMEPULSE: no longer names the net of U1.29 (GPIO18)
- no-connect marks 12 -> 14
Changed lines of the file:
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@@
   )
   (no_connect (at 41.91 50.8))
+  (no_connect (at 101.6 233.68))
   (no_connect (at 228.6 256.54))
   (no_connect (at 152.4 231.14))
@@
   (no_connect (at 228.6 259.08))
   (no_connect (at 41.91 53.34))
+  (no_connect (at 101.6 231.14))
   (no_connect (at 101.6 243.84))
   (wire (pts (xy 110.49 165.1) (xy 110.49 166.37))
@@
     (stroke (width 0) (type default))
   )
+  (wire (pts (xy 129.54 243.84) (xy 129.54 245.11))
+    (stroke (width 0) (type default))
+  )
   (wire (pts (xy 245.11 204.47) (xy 257.81 204.47))
     (stroke (width 0) (type default))
@@
     (stroke (width 0) (type default))
   )
+  (wire (pts (xy 101.6 238.76) (xy 130.81 238.76))
+    (stroke (width 0) (type default))
+  )
   (wire (pts (xy 359.41 78.74) (xy 359.41 77.47))
     (stroke (width 0) (type default))
@@
     (stroke (width 0) (type default))
   )
+  (wire (pts (xy 101.6 241.3) (xy 130.81 241.3))
+    (stroke (width 0) (type default))
+  )
   (wire (pts (xy 289.56 55.88) (xy 297.18 55.88))
     (stroke (width 0) (type default))
@@
     (stroke (width 0) (type default))
   )
+  (wire (pts (xy 129.54 236.22) (xy 129.54 234.95))
+    (stroke (width 0) (type default))
+  )
   (polyline (pts (xy 209.55 283.21) (xy 265.43 283.21))
     (stroke (width 0) (type dash))
@@
     (stroke (width 0) (type default))
   )
+  (wire (pts (xy 130.81 243.84) (xy 129.54 243.84))
+    (stroke (width 0) (type default))
+  )
   (polyline (pts (xy 233.68 21.59) (xy 323.85 21.59))
     (stroke (width 0) (type dash))
@@
     (stroke (width 0) (type default))
   )
-  (wire (pts (xy 101.6 233.68) (xy 123.19 233.68))
-    (stroke (width 0) (type default))
-  )
   (wire (pts (xy 214.63 185.42) (xy 214.63 186.69))
     (stroke (width 0) (type default))
@@
     (stroke (width 0) (type default))
   )
+  (wire (pts (xy 130.81 236.22) (xy 129.54 236.22))
+    (stroke (width 0) (type default))
+  )
   (wire (pts (xy 242.57 67.31) (xy 242.57 68.58))
     (stroke (width 0) (type default))
@@
     (stroke (width 0) (type default))
   )
-  (wire (pts (xy 101.6 241.3) (xy 123.19 241.3))
-    (stroke (width 0) (type default))
-  )
-  (wire (pts (xy 101.6 238.76) (xy 123.19 238.76))
-    (stroke (width 0) (type default))
-  )
   (wire (pts (xy 87.63 87.63) (xy 87.63 88.9))
     (stroke (width 0) (type default))
@@
     (stroke (width 0) (type default))
   )
-  (wire (pts (xy 101.6 231.14) (xy 123.19 231.14))
-    (stroke (width 0) (type default))
-  )
   (wire (pts (xy 161.29 59.69) (xy 186.69 59.69))
     (stroke (width 0) (type default))
@@
     (effects (font (size 1.27 1.27)) (justify left bottom))
   )
-  (label "EXTINT" (at 123.19 231.14 180) (fields_autoplaced)
-    (effects (font (size 1.27 1.27)) (justify right bottom))
-  )
-  (label "TIMEPULSE" (at 123.19 233.68 180) (fields_autoplaced)
-    (effects (font (size 1.27 1.27)) (justify right bottom))
-  )
   (label "MISO" (at 261.62 261.62 180) (fields_autoplaced)
     (effects (font (size 1.27 1.27)) (justify right bottom))
@@
     (pin "4")
     (pin "5")
-    (pin "EP")
     (pin "6")
+    (pin "EP")
     (instances
       (project "Babel_Fish"
@@
     )
   )
+  (symbol (lib_id "Connector_Generic:Conn_01x04") (at 135.89 238.76 0) (unit 1)
+    (in_bom yes) (on_board yes) (dnp no) (fields_autoplaced)
+    (property "Reference" "J5" (at 138.43 238.76 0)
+      (effects (font (size 1.27 1.27)) (justify left))
+    )
+    (property "Value" "Conn_01x04" (at 138.43 241.3 0)
+      (effects (font (size 1.27 1.27)) (justify left))
+    )
+    (property "Footprint" "Connector_PinHeader_2.54mm:PinHeader_1x04_P2.54mm_Vertical" (at 135.89 238.76 0)
+      (effects (font (size 1.27 1.27)) hide)
+    )
+    (property "Datasheet" "~" (at 135.89 238.76 0)
+      (effects (font (size 1.27 1.27)) hide)
+    )
+    (pin "1")
+    (pin "2")
+    (pin "3")
+    (pin "4")
+    (instances
+      (project "Babel_Fish"
+        (path "/1251a41c-aa26-471e-a374-8838d59fff79"
+          (reference "J5") (unit 1)
+        )
+      )
+    )
+  )
   (symbol (lib_id "BITSv5:MCU_RaspberryPi_RP2040") (at 69.85 220.98 0) (unit 1)
     (in_bom yes) (on_board yes) (dnp no)
@@
     )
   )
+  (symbol (lib_id "power:+3V3") (at 129.54 234.95 0) (unit 1)
+    (in_bom yes) (on_board yes) (dnp no)
+    (property "Reference" "#PWR053" (at 129.54 238.76 0)
+      (effects (font (size 1.27 1.27)) hide)
+    )
+    (property "Value" "+3V3" (at 129.54 231.14 0)
+      (effects (font (size 1.27 1.27)))
+    )
+    (property "Footprint" "" (at 129.54 234.95 0)
+      (effects (font (size 1.27 1.27)) hide)
+    )
+    (property "Datasheet" "" (at 129.54 234.95 0)
+      (effects (font (size 1.27 1.27)) hide)
+    )
+    (pin "1")
+    (instances
+      (project "Babel_Fish"
+        (path "/1251a41c-aa26-471e-a374-8838d59fff79"
+          (reference "#PWR053") (unit 1)
+        )
+      )
+    )
+  )
   (symbol (lib_id "power:GND") (at 271.78 81.28 0) (unit 1)
     (in_bom yes) (on_board yes) (dnp no)
@@
     )
   )
+  (symbol (lib_id "power:GND") (at 129.54 245.11 0) (unit 1)
+    (in_bom yes) (on_board yes) (dnp no)
+    (property "Reference" "#PWR052" (at 129.54 251.46 0)
+      (effects (font (size 1.27 1.27)) hide)
+    )
+    (property "Value" "GND" (at 129.54 248.92 0)
+      (effects (font (size 1.27 1.27)))
+    )
+    (property "Footprint" "" (at 129.54 245.11 0)
+      (effects (font (size 1.27 1.27)) hide)
+    )
+    (property "Datasheet" "" (at 129.54 245.11 0)
+      (effects (font (size 1.27 1.27)) hide)
+    )
+    (pin "1")
+    (instances
+      (project "Babel_Fish"
+        (path "/1251a41c-aa26-471e-a374-8838d59fff79"
+          (reference "#PWR052") (unit 1)
+        )
+      )
+    )
+  )
   (symbol (lib_id "power:+3V3") (at 33.02 218.44 0) (unit 1)
     (in_bom yes) (on_board yes) (dnp no)
@@
     (pin "3")
     (pin "4")
-    (pin "9")
     (pin "5")
     (pin "6")
     (pin "7")
     (pin "8")
+    (pin "9")
     (instances
       (project "Babel_Fish"
